File: power distribution board/v3/pdb.kicad_pcb (KiCad board)
At the start: 2 copper layers, 77.5 x 85.1 mm, 24 parts, among them J1 Conn_01x04, J10 Conn_01x04, J11 Conn_01x04, J12 Conn_01x04, J13 Conn_01x04, J14 Conn_01x04, J15 Conn_01x04, J16 Conn_01x04, J17 Conn_02x20_Odd_Even, J18 Conn_02x20_Odd_Even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

Commit message: Tweaks to the layout.
Routing:
- net /D10: track 57.1 -> 59.7 mm
- net /D9: track 70.1 -> 71.2 mm
